File: a500_1mb_backdoor_ram.kicad_sch (KiCad schematic)
At the start: 20 parts, among them J1 Expansion, U1 V53C181608K60, U2 V53C181608K60

Commit message: Version 2.0 - fixing GND vs. VDD connection
Parts:
- added C3, C4: 100n, Capacitor_SMD:C_0402_1005Metric, symbol Device:C
Connections:
- net +5V: now also C3.1, C4.1; no longer J1.21 (Pin_21), J1.22 (Pin_22)
- net GND: now also J1.21 (Pin_21), J1.22 (Pin_22), C3.2, C4.2
